File: Adapter_KiCad/lofence.kicad_sch (KiCad schematic)
At the start: 25 parts, among them J1 Fence+, J2 Fence-, U1 Opamp_Dual_Generic

Commit message: First changes in KiCad
Parts:
- added U2: WIFI_KIT_32__V3_, WIFI_KIT_32__V3:MODULE_WIFI_KIT_32__V3_, symbol WIFI_KIT_32__V3_:WIFI_KIT_32__V3_
Connections:
- new net +3.3V: U2.J3_11 (GPIO37/SPIDQS/FSPIQ/SUBSPIQ/ADC_CTRL)
- new net 3V3: U2.J3_2 (3V3), U2.J3_3 (3V3)
- new net VE: U2.J2_3 (VE), U2.J2_4 (VE)

Commit message: Finished PCB & Schematic
Parts:
- removed C5, C7: 100nF, Capacitors_SMD:C_0805_HandSoldering, symbol Device:C
- removed D2, D8: BAV70LT, TO_SOT_Packages_SMD:SOT-23, symbol lofence-rescue:BAV70LT-kiu
- removed MH1, MH2, MH3, MH4, MH5, MH6: MountingHole, Mounting_Holes:MountingHole_2.7mm_M2.5, symbol Mechanical:MountingHole
- removed R10, R16, R17, R18, R7: 100k, Resistors_SMD:R_0805_HandSoldering, symbol Device:R
- removed R12, R19: 1M, Resistors_SMD:R_0805_HandSoldering, symbol Device:R
- removed U1: Opamp_Dual_Generic, Housings_SOIC:SOIC-8_3.9x4.9mm_Pitch1.27mm, symbol lofence-rescue:Opamp_Dual_Generic-Device
- added D1: SMAJ5.0CA, Diode_SMD:D_SMA, symbol Diode:SMAJ5.0CA
- added D2: BAT54S, Package_TO_SOT_SMD:SOT-23, symbol Diode:BAT54S
- added R5: 10k, Resistor_SMD:R_0805_2012Metric_Pad1.20x1.40mm_HandSolder, symbol Device:R
- added R6: 1M, Resistor_SMD:R_0805_2012Metric_Pad1.20x1.40mm_HandSolder, symbol Device:R
- C1: footprint Capacitors_SMD:C_0805_HandSoldering -> Capacitor_SMD:C_0805_2012Metric_Pad1.18x1.45mm_HandSolder
- R1, R2: footprint Resistors_ThroughHole:R_Axial_DIN0516_L15.5mm_D5.0mm_P20.32mm_Horizontal -> Resistor_THT:R_Axial_DIN0414_L11.9mm_D4.5mm_P15.24mm_Horizontal
- R3: footprint Resistors_ThroughHole:R_Axial_DIN0207_L6.3mm_D2.5mm_P10.16mm_Horizontal -> Resistor_SMD:R_1206_3216Metric_Pad1.30x1.75mm_HandSolder
- R4: value 5k8 -> 5k1; footprint Resistors_SMD:R_0805_HandSoldering -> Resistor_SMD:R_0805_2012Metric_Pad1.20x1.40mm_HandSolder
Connections:
- net 3V3 is gone; now on net +3.3V: U2.J3_2 (3V3), U2.J3_3 (3V3)
- net ADC_POWER is gone; now on net ADC_FENCE: C1.1
- net +3.3V: now also U2.J3_4 (GPIO37/SPIDQS/FSPIQ/SUBSPIQ/ADC_Ctrl), D2.2 (K); no longer U2.J3_11 (GPIO37/SPIDQS/FSPIQ/SUBSPIQ/ADC_CTRL)
- net GND: now also U2.J2_1 (GND_J2), U2.J3_1 (GND_J3), D1.1 (A1), D2.1 (A), R6.1
- net ADC_FENCE: now reaches U2.J3_13 (GPIO2/ADC1_CH1/TOUCH2)
- net ADC_FENCE: now also D2.3 (COM), R5.1, R6.2
- net +5V: now reaches U2.J2_2 (5V)
- net PROBE: no longer names the net of R3.1, R4.2
- net PROBE: now also D1.2 (A2), R5.2
- net VE: no longer names the net of U2.J2_3 (VE/OUTPUT_3.3V)
- net VE: no longer U2.J2_4 (VE)
Other:
- note removed: "AMP+"
- note removed: "Amp-"
- note removed: "Mechanics"
- note removed: "Power OpAmp"
- moved on the sheet: J1, J2, R1, R2, R3, R4
